Commit message: wheels added

File: src/cube_description/urdf/object.urdf (robot description, URDF)
Before this commit: robot simple_box, 1 links, 0 joints
Links:
- added link inertia_wheel_roll, mass 0.5; collision cylinder length=0.01 radius=0.08; visual cylinder length=0.01 radius=0.08
Joints:
- added joint inertia_wheel_roll_joint: type continuous, parent my_box, child inertia_wheel_roll, origin xyz=0.1 0.0 0.0 rpy=0 1.57 0, axis 0 0 1, limit effort=200 velocity=1000.0

Commit message: co-ordinate frame conversion done from unity to gazebo

File: src/cube_description/urdf/object.urdf (robot description, URDF)
Before this commit: robot simple_box, 2 links, 1 joints
Links:
- removed link inertia_wheel_roll
- added link world
Joints:
- removed joint inertia_wheel_roll_joint
- added joint base: type continuous, parent world, child my_box, origin xyz=0 0 1, axis 0 0 -1

Commit message: gazebo cube mimics unity

File: src/cube_description/urdf/object.urdf (robot description, URDF)
Before this commit: robot simple_box, 2 links, 1 joints
Links:
- removed link world
Joints:
- removed joint base
